File: omsdr.sch (KiCad schematic (older format))
At the start: 52 parts, among them J1 I/Q Out, J2 ANT, J3 ISP, J4 LO, J8 PWR, SW1 SW_SPST, SW2 SW_SPST, T1 CX2074NL, U1 LT6231, U2 FST3253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

Commit message: Replace 3.3 V regul L78L33ABUTR with LDK320ADU33R
Almost same price, lower noise, better PSSR and slightly better
pinout. Same SOT-89 package. Chances in schematic and PCB.
Parts:
- removed U3: L78L33ABUTR, TO_SOT_Packages_SMD:SOT-89-3_Handsoldering, symbol regul:AP2204RB-5.0
- added U3: LDK320ADU33R, TO_SOT_Packages_SMD:SOT-89-3_Handsoldering, symbol regul:MCP1703A-3302_SOT89
Changed lines of the file:
@@
 SCK
-$Comp
-L regul:AP2204RB-5.0 U3
-U 1 1 5A059921
-P 1700 4800
-F 0 "U3" H 1700 5042 50  0000 C CNN
-F 1 " L78L33ABUTR " H 1700 4951 50  0000 C CNN
-F 2 "TO_SOT_Packages_SMD:SOT-89-3_Handsoldering" H 1700 5025 50  0001 C CNN
-F 3 "" H 1700 4800 50  0001 C CNN
-F 4 "DIST DIGIEKY 497-7286-1-ND" H 1700 4800 60  0001 C CNN "BOM"
-	1    1700 4800
-	1    0    0    -1
-$EndComp
 $Comp
 L power:GND #PWR024
@@
 NoConn ~ 4850 5800
 NoConn ~ 4850 5700
+$Comp
+L regul:MCP1703A-3302_SOT89 U3
+U 1 1 5A5FA826
+P 1700 4800
+F 0 "U3" H 1700 5042 50  0000 C CNN
+F 1 "LDK320ADU33R" H 1700 4951 50  0000 C CNN
+F 2 "TO_SOT_Packages_SMD:SOT-89-3_Handsoldering" H 1700 5000 50  0001 C CNN
+F 3 "" H 1700 4750 50  0001 C CNN
+F 4 "DIST DIGIKEY 497-17585-1-ND" H 1700 4800 50  0001 C CNN "BOM"
+	1    1700 4800
+	1    0    0    -1
+$EndComp
 $EndSCHEMATC

Commit message: Changed sample cap loading resistor frorm 10 Ohms to 49.9 Ohms
Parts:
- R4, R9: value 10 -> 49.9
Changed lines of the file:
@@
 P 8400 3750
 F 0 "R4" V 8300 3750 50  0000 C CNN
-F 1 "10" V 8400 3750 50  0000 C CNN
+F 1 "49.9" V 8400 3750 50  0000 C CNN
 F 2 "Resistors_SMD:R_1206_HandSoldering" V 8330 3750 50  0001 C CNN
 F 3 "" H 8400 3750 50  0001 C CNN
@@
 P 8400 2350
 F 0 "R9" V 8300 2350 50  0000 C CNN
-F 1 "10" V 8400 2350 50  0000 C CNN
+F 1 "49.9" V 8400 2350 50  0000 C CNN
 F 2 "Resistors_SMD:R_1206_HandSoldering" V 8330 2350 50  0001 C CNN
 F 3 "" H 8400 2350 50  0001 C CNN

Commit message: Component values for opamp feedback network
Parts:
- C10, C13: value C -> 390p
- R10, R7: value R -> 4.99k
Changed lines of the file:
@@
 P 8950 4350
 F 0 "R7" V 8850 4350 50  0000 C CNN
-F 1 "R" V 8950 4350 50  0000 C CNN
+F 1 "4.99k" V 8950 4350 50  0000 C CNN
 F 2 "Resistors_SMD:R_1206_HandSoldering" V 8880 4350 50  0001 C CNN
 F 3 "" H 8950 4350 50  0001 C CNN
@@
 U 1 1 5A04F551
 P 8950 4550
-F 0 "C10" V 9000 4650 50  0000 C CNN
-F 1 "C" V 8900 4450 50  0000 C CNN
+F 0 "C10" V 9000 4700 50  0000 C CNN
+F 1 "390p" V 8900 4400 50  0000 C CNN
 F 2 "Capacitors_SMD:C_1206_HandSoldering" H 8988 4400 50  0001 C CNN
 F 3 "" H 8950 4550 50  0001 C CNN
@@
 P 8900 2900
 F 0 "R10" V 8800 2900 50  0000 C CNN
-F 1 "R" V 8900 2900 50  0000 C CNN
+F 1 "4.99k" V 8900 2900 50  0000 C CNN
 F 2 "Resistors_SMD:R_1206_HandSoldering" V 8830 2900 50  0001 C CNN
 F 3 "" H 8900 2900 50  0001 C CNN
@@
 U 1 1 5A04FEE6
 P 8900 3100
-F 0 "C13" V 8950 3200 50  0000 C CNN
-F 1 "C" V 8850 3000 50  0000 C CNN
+F 0 "C13" V 8950 3250 50  0000 C CNN
+F 1 "390p" V 8850 2950 50  0000 C CNN
 F 2 "Capacitors_SMD:C_1206_HandSoldering" H 8938 2950 50  0001 C CNN
 F 3 "" H 8900 3100 50  0001 C CNN

Commit message: Multiplexer chip EOL, replaced with substitute order number
Parts:
- U2: BOM DIST DIGIKEY FST3253MXFSCT-ND -> DIST DIGIKEY 296-19206-1-ND
Changed lines of the file:
@@
 F 2 "IPC7351-Most:SOIC127P600X180-16" H 6950 1900 50  0001 C CNN
 F 3 "https://www.fairchildsemi.com/datasheets/FS/FST3253.pdf" H 6950 1700 50  0001 C CNN
-F 4 "DIST DIGIKEY FST3253MXFSCT-ND" H 6950 1800 60  0001 C CNN "BOM"
+F 4 "DIST DIGIKEY 296-19206-1-ND" H 6950 1800 60  0001 C CNN "BOM"
 	1    6950 2800
 	-1   0    0    -1

Commit message: Adding more component values and BOM digikey order numbers
Parts:
- C1, C12, C3: symbol device:C -> Device:C; BOM (none) -> CAP MLCC 0.1u ±10% ≥X7R [1206]
- C10, C13: symbol device:C -> Device:C; BOM (none) -> CAP MLCC 390p ±5% NP0 [1206]
- C11, C2, C5: BOM (none) -> CAP MLCC 0.1u ±10% ≥X7R [1206]
- C14: BOM (none) -> CAP MLCC 4.7u ±20% 10V [1206]
- C16, C4: symbol device:C -> Device:C; BOM (none) -> CAP MLCC 4.7u ±20% 10V [1206]
- C6: value C -> 110p; BOM (none) -> CAP MLCC 110p ±5% NP0 [1206]
- C7, C9: BOM (none) -> CAP MLCC 0.047u ±10% ≥X5R [1206]
- C8: value C -> 1500p; BOM (none) -> CAP MLCC 1500p ±5% NP0 [1206]
- D1, D2, D3, D4: BOM (none) -> DIST DIGIKEY 732-4984-1-ND
- J2: BOM (none) -> DIST DIGIKEY CON-SMA-EDGE-S-ND
- J3: symbol Connector:Conn_02x03_Odd_Even -> Connector_Generic:Conn_02x03_Odd_Even; BOM (none) -> DIST DIGIKEY 609-2846-ND
- J8: symbol Connector:Conn_01x05 -> Connector_Generic:Conn_01x05; BOM (none) -> DIST DIGIKEY S1012EC-05-ND
- L1: value L -> 4.7u; BOM (none) -> DIST DIGIKEY 587-2034-1-ND
- R1, R2: BOM (none) -> RES SMD 1k 1% [1206]
- R10, R7: symbol device:R -> Device:R; BOM (none) -> RES SMD 4.99k 1% [1206]
- R11, R12, R13, R14: BOM (none) -> RES SMD 1k 1% [0805]
- R3, R8: BOM (none) -> RES SMD 100 1% [1206]
- R4, R9: BOM (none) -> RES SMD 49.9 1% [1206]
- R5, R6: symbol device:R -> Device:R; BOM (none) -> RES SMD 10 1% [1206]
- SW1, SW2: BOM (none) -> DIST DIGIKEY EG2531CT-ND
- U1: BOM (none) -> DIST DIGIKEY LT6231CS8#PBF-ND
- U5: BOM (none) -> DIST DIGIKEY ATTINY24A-SSU-ND

Commit message: Changes due to new kicad version (library upgrades etc.)
Parts:
- C11, C14, C2, C5, C6, C7, C8, C9: symbol device:C -> Device:C
- D1, D2, D3, D4: symbol device:LED -> Device:LED
- J1: symbol Connector:Audio-Jack-3 -> omsdr-rescue:Audio-Jack-3-Connector
- J4: symbol Connector:Conn_01x03 -> Connector_Generic:Conn_01x03
- L1: symbol device:L -> Device:L
- MH1, MH2, MH3, MH4: symbol Mechanical:Mounting_Hole_PAD -> Mechanical:MountingHole_Pad
- R1, R11, R12, R13, R14, R2, R3, R4, R8, R9: symbol device:R -> Device:R
- T1: symbol device:Transformer_1P_SS -> Device:Transformer_1P_SS
- U1: symbol linear:LT6233 -> omsdr-rescue:LT6233-linear
- U2: symbol onsemi:FST3253 -> omsdr-rescue:FST3253-onsemi
- U3: symbol regul:MCP1703A-3302_SOT89 -> Regulator_Linear:MCP1703A-3302_SOT89
- U4: symbol omsdr-rescue:Si5351A-RESCUE-omsdr -> silabs:Si5351A
- U5: symbol atmel:ATTINY24-20SSU -> omsdr-rescue:ATTINY24-20SSU-atmel
- X1: symbol device:Crystal_Small -> Device:Crystal_Small
Changed lines of the file:
@@
 $EndComp
 $Comp
-L device:C C6
+L Device:C C6
 U 1 1 5A049F14
 P 1650 2450
@@
 $EndComp
 $Comp
-L device:C C8
+L Device:C C8
 U 1 1 5A049F8F
 P 2500 2650
@@
 $EndComp
 $Comp
-L device:L L1
+L Device:L L1
 U 1 1 5A04A010
 P 2150 2450
@@
 $EndComp
 $Comp
-L device:Transformer_1P_SS T1
+L Device:Transformer_1P_SS T1
 U 1 1 5A04A23A
 P 3300 2650
@@
 	2000 2450 1800 2450
 Wire Wire Line
-	1500 2450 1150 2450
-Wire Wire Line
 	1000 2650 1000 2900
 $Comp
-L onsemi:FST3253 U2
+L omsdr-rescue:FST3253-onsemi U2
 U 1 1 5A04A0A1
 P 6950 2800
@@
 	2500 2800 2500 2900
 $Comp
-L device:R R1
+L Device:R R1
 U 1 1 5A04A538
 P 4200 1650
@@
 $EndComp
 $Comp
-L device:R R2
+L Device:R R2
 U 1 1 5A04A5AB
 P 4200 2050
@@
 	3700 2850 5650 2850
 $Comp
-L linear:LT6233 U1
+L omsdr-rescue:LT6233-linear U1
 U 1 1 5A04AECD
 P 9050 3650
@@
 Vhalf
 $Comp
-L device:R R4
+L Device:R R4
 U 1 1 5A04CCC8
 P 8400 3750
@@
 $EndComp
 $Comp
-L device:R R9
+L Device:R R9
 U 1 1 5A04CE0B
 P 8400 2350
@@
 	8550 2350 8600 2350
 $Comp
-L device:C C2
+L Device:C C2
 U 1 1 5A04D20D
 P 9150 1800
@@
 Connection ~ 6250 2850
 $Comp
-L omsdr-rescue:Si5351A-RESCUE-omsdr U4
+L silabs:Si5351A U4
 U 1 1 5A0528DB
 P 6900 5050
@@
 NoConn ~ 7500 5000
 $Comp
-L device:Crystal_Small X1
+L Device:Crystal_Small X1
 U 1 1 5A052EA0
 P 7700 5200
@@
 	1700 5100 1700 5150
 $Comp
-L device:C C14
+L Device:C C14
 U 1 1 5A05A413
 P 1000 4950
@@
 Connection ~ 6200 4800
 $Comp
-L device:C C9
+L Device:C C9
 U 1 1 5A05507D
 P 8000 2500
@@
 $EndComp
 $Comp
-L device:C C7
+L Device:C C7
 U 1 1 5A05515B
 P 8000 3100
@@
 Connection ~ 8000 2950
 $Comp
-L device:C C5
+L Device:C C5
 U 1 1 5A0576CE
 P 9600 3650
@@
 $EndComp
 $Comp
-L device:C C11
+L Device:C C11
 U 1 1 5A05777E
 P 9600 2250
@@
 $EndComp
 $Comp
-L device:R R3
+L Device:R R3
 U 1 1 5A0578C6
 P 10000 3650
@@
 $EndComp
 $Comp
-L device:R R8
+L Device:R R8
 U 1 1 5A057990
 P 10000 2250
@@
 	10150 3650 10400 3650
 $Comp
-L Mechanical:Mounting_Hole_PAD MH1
+L Mechanical:MountingHole_Pad MH1
 U 1 1 5A0577BA
 P 1400 6900
@@
 $EndComp
 $Comp
-L Mechanical:Mounting_Hole_PAD MH2
+L Mechanical:MountingHole_Pad MH2
 U 1 1 5A057FC9
 P 1800 6900
@@
 $EndComp
 $Comp
-L Mechanical:Mounting_Hole_PAD MH3
+L Mechanical:MountingHole_Pad MH3
 U 1 1 5A0580BB
 P 2200 6900
@@
 $EndComp
 $Comp
-L Mechanical:Mounting_Hole_PAD MH4
+L Mechanical:MountingHole_Pad MH4
 U 1 1 5A0580C1
 P 2600 6900
@@
 $EndComp
 $Comp
-L device:LED D1
+L Device:LED D1
 U 1 1 5A06BFEC
 P 3650 4100
@@
 $EndComp
 $Comp
-L device:R R11
+L Device:R R11
 U 1 1 5A06C30F
 P 3650 3800
@@
 $EndComp
 $Comp
-L device:LED D2
+L Device:LED D2
 U 1 1 5A06CB4A
 P 4100 4100
@@
 $EndComp
 $Comp
-L device:R R12
+L Device:R R12
 U 1 1 5A06CB50
 P 4100 3800
@@
 $EndComp
 $Comp
-L device:LED D3
+L Device:LED D3
 U 1 1 5A06CCB4
 P 4500 4100
@@
 $EndComp
 $Comp
-L device:R R13
+L Device:R R13
 U 1 1 5A06CCBA
 P 4500 3800
@@
 $EndComp
 $Comp
-L device:LED D4
+L Device:LED D4
 U 1 1 5A06CCC6
 P 4950 4100
@@
 $EndComp
 $Comp
-L device:R R14
+L Device:R R14
 U 1 1 5A06CCCC
 P 4950 3800
@@
 Connection ~ 6350 7000
 $Comp
-L linear:LT6233 U1
+L omsdr-rescue:LT6233-linear U1
 U 2 1 5A06216D
 P 9000 2250
@@
 $EndComp
 $Comp
-L Connector:Conn_01x03 J4
+L Connector_Generic:Conn_01x03 J4
 U 1 1 5A069F9E
 P 8100 4150
@@
 Connection ~ 7750 4050
 $Comp
-L Connector:Audio-Jack-3 J1
+L omsdr-rescue:Audio-Jack-3-Connector J1
 U 1 1 5A050DB8
 P 10600 2250
@@
 	5050 6000 4850 6000
 $Comp
-L atmel:ATTINY24-20SSU U5
+L omsdr-rescue:ATTINY24-20SSU-atmel U5
 U 1 1 5A5637E0
 P 3800 5400
@@
 NoConn ~ 4850 5700
 $Comp
-L regul:MCP1703A-3302_SOT89 U3
+L Regulator_Linear:MCP1703A-3302_SOT89 U3
 U 1 1 5A5FA826
 P 1700 4800
@@
 	1    0    0    -1
 $EndComp
+Wire Wire Line
+	1200 2450 1500 2450
 $EndSCHEMATC

Commit message: Use FST3253 from kicad-schlib instead of cached
Parts:
- U2: symbol omsdr-rescue:FST3253-onsemi -> onsemi:FST3253
Changed lines of the file:
@@
 	1000 2650 1000 2900
 $Comp
-L omsdr-rescue:FST3253-onsemi U2
+L onsemi:FST3253 U2
 U 1 1 5A04A0A1
 P 6950 2800

Commit message: Replacing SMA connector since the one used was phased out from kicad
No BOM as we are better off ordering this from China
Parts:
- J2: footprint Connectors_Molex:Molex_SMA_Jack_Edge_Mount -> Connector_Coaxial:SMA_Amphenol_132289_EdgeMount; BOM DIST DIGIKEY CON-SMA-EDGE-S-ND -> (none)
Changed lines of the file:
@@
 F 0 "J2" H 1100 2426 50  0000 L CNN
 F 1 "ANT" H 1100 2335 50  0000 L CNN
-F 2 "Connectors_Molex:Molex_SMA_Jack_Edge_Mount" H 1000 2450 50  0001 C CNN
+F 2 "Connector_Coaxial:SMA_Amphenol_132289_EdgeMount" H 1000 2450 50  0001 C CNN
 F 3 "" H 1000 2450 50  0001 C CNN
-F 4 "DIST DIGIKEY CON-SMA-EDGE-S-ND " H 1000 2450 50  0001 C CNN "BOM"
 	1    1000 2450
 	-1   0    0    -1
