File: omsdr.sch (KiCad schematic (older format))
At the start: 52 parts, among them J1 I/Q Out, J2 ANT, J3 ISP, J4 LO, J8 PWR, SW1 SW_SPST, SW2 SW_SPST, T1 CX2074NL, U1 LT6231, U2 FST3253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

Commit message: Changed my mind: Swapped SMA edge connector for smaller version
Parts:
- J2: footprint Connector_Coaxial:SMA_Amphenol_132289_EdgeMount -> local:SMA_edge_mount_small
Changed lines of the file:
@@
 F 0 "J2" H 1100 2426 50  0000 L CNN
 F 1 "ANT" H 1100 2335 50  0000 L CNN
-F 2 "Connector_Coaxial:SMA_Amphenol_132289_EdgeMount" H 1000 2450 50  0001 C CNN
+F 2 "local:SMA_edge_mount_small" H 1000 2450 50  0001 C CNN
 F 3 "" H 1000 2450 50  0001 C CNN
 	1    1000 2450

Commit message: Reworked input bandpass filter
Parts:
- added L2: 0.56u, Inductor_SMD:L_0805_2012Metric_Pad1.15x1.40mm_HandSolder, symbol Device:L
- C6: footprint Capacitors_SMD:C_1206_HandSoldering -> Capacitor_SMD:C_1206_3216Metric_Pad1.42x1.75mm_HandSolder
- C8: value 1500p -> 680p; footprint Capacitors_SMD:C_1206_HandSoldering -> Capacitor_SMD:C_1206_3216Metric_Pad1.42x1.75mm_HandSolder; BOM CAP MLCC 1500p ±5% NP0 [1206] -> CAP MLCC 680p ±5% NP0 [1206]
- L1: footprint Resistors_SMD:R_1206_HandSoldering -> Inductor_SMD:L_1206_3216Metric_Pad1.42x1.75mm_HandSolder
Connections:
- wire segments 135 -> 136
Changed lines of the file:
@@
 L Device:C C6
 U 1 1 5A049F14
-P 1650 2450
-F 0 "C6" V 1500 2450 50  0000 C CNN
-F 1 "110p" V 1800 2450 50  0000 C CNN
-F 2 "Capacitors_SMD:C_1206_HandSoldering" H 1688 2300 50  0001 C CNN
-F 3 "" H 1650 2450 50  0001 C CNN
-F 4 "CAP MLCC 110p ±5% NP0 [1206]" V 1650 2450 50  0001 C CNN "BOM"
-	1    1650 2450
+P 1450 2450
+F 0 "C6" V 1300 2450 50  0000 C CNN
+F 1 "110p" V 1600 2450 50  0000 C CNN
+F 2 "Capacitor_SMD:C_1206_3216Metric_Pad1.42x1.75mm_HandSolder" H 1488 2300 50  0001 C CNN
+F 3 "" H 1450 2450 50  0001 C CNN
+F 4 "CAP MLCC 110p ±5% NP0 [1206]" V 1450 2450 50  0001 C CNN "BOM"
+	1    1450 2450
 	0    1    1    0
 $EndComp
@@
 L Device:C C8
 U 1 1 5A049F8F
-P 2500 2650
-F 0 "C8" H 2615 2696 50  0000 L CNN
-F 1 "1500p" H 2615 2605 50  0000 L CNN
-F 2 "Capacitors_SMD:C_1206_HandSoldering" H 2538 2500 50  0001 C CNN
-F 3 "" H 2500 2650 50  0001 C CNN
-F 4 "CAP MLCC 1500p  ±5% NP0 [1206]" H 2500 2650 50  0001 C CNN "BOM"
-	1    2500 2650
+P 2150 2700
+F 0 "C8" H 2265 2746 50  0000 L CNN
+F 1 "680p" H 2265 2655 50  0000 L CNN
+F 2 "Capacitor_SMD:C_1206_3216Metric_Pad1.42x1.75mm_HandSolder" H 2188 2550 50  0001 C CNN
+F 3 "" H 2150 2700 50  0001 C CNN
+F 4 "CAP MLCC 680p  ±5% NP0 [1206]" H 2150 2700 50  0001 C CNN "BOM"
+	1    2150 2700
 	1    0    0    -1
 $EndComp
@@
 L Device:L L1
 U 1 1 5A04A010
-P 2150 2450
-F 0 "L1" V 1972 2450 50  0000 C CNN
-F 1 "4.7u" V 2300 2450 50  0000 C CNN
-F 2 "Resistors_SMD:R_1206_HandSoldering" H 2150 2450 50  0001 C CNN
-F 3 "" H 2150 2450 50  0001 C CNN
-F 4 "DIST DIGIKEY  587-2034-1-ND" V 2150 2450 50  0001 C CNN "BOM"
-	1    2150 2450
+P 1850 2450
+F 0 "L1" V 1672 2450 50  0000 C CNN
+F 1 "4.7u" V 2000 2450 50  0000 C CNN
+F 2 "Inductor_SMD:L_1206_3216Metric_Pad1.42x1.75mm_HandSolder" H 1850 2450 50  0001 C CNN
+F 3 "" H 1850 2450 50  0001 C CNN
+F 4 "DIST DIGIKEY  587-2034-1-ND" V 1850 2450 50  0001 C CNN "BOM"
+	1    1850 2450
 	0    1    1    0
 $EndComp
@@
 L power:GND #PWR02
 U 1 1 5A04A0B8
-P 2500 2900
-F 0 "#PWR02" H 2500 2650 50  0001 C CNN
-F 1 "GND" H 2505 2727 50  0000 C CNN
-F 2 "" H 2500 2900 50  0001 C CNN
-F 3 "" H 2500 2900 50  0001 C CNN
-	1    2500 2900
+P 2150 2900
+F 0 "#PWR02" H 2150 2650 50  0001 C CNN
+F 1 "GND" H 2155 2727 50  0000 C CNN
+F 2 "" H 2150 2900 50  0001 C CNN
+F 3 "" H 2150 2900 50  0001 C CNN
+	1    2150 2900
 	1    0    0    -1
 $EndComp
@@
 	2900 2900 2900 2850
 Wire Wire Line
-	2300 2450 2500 2450
-Wire Wire Line
-	2500 2450 2500 2500
-Connection ~ 2500 2450
-Wire Wire Line
-	2000 2450 1800 2450
+	2000 2450 2150 2450
+Wire Wire Line
+	2150 2450 2150 2550
+Wire Wire Line
+	1700 2450 1600 2450
 Wire Wire Line
 	1000 2650 1000 2900
@@
 $EndComp
 Wire Wire Line
-	2500 2800 2500 2900
+	2150 2850 2150 2900
 $Comp
 L Device:R R1
@@
 	10800 2150 10950 2150
 Wire Wire Line
-	2500 2450 2900 2450
-Wire Wire Line
 	4200 1850 4200 1900
 Wire Wire Line
@@
 $EndComp
 Wire Wire Line
-	1200 2450 1500 2450
+	1200 2450 1300 2450
+$Comp
+L Device:L L2
+U 1 1 5C8E7AFF
+P 2550 2450
+F 0 "L2" V 2372 2450 50  0000 C CNN
+F 1 "0.56u" V 2700 2450 50  0000 C CNN
+F 2 "Inductor_SMD:L_0805_2012Metric_Pad1.15x1.40mm_HandSolder" H 2550 2450 50  0001 C CNN
+F 3 "" H 2550 2450 50  0001 C CNN
+F 4 "DIST DIGIKEY  LBM2016TR56J" V 2550 2450 50  0001 C CNN "BOM"
+	1    2550 2450
+	0    1    1    0
+$EndComp
+Wire Wire Line
+	2900 2450 2700 2450
+Wire Wire Line
+	2400 2450 2150 2450
+Connection ~ 2150 2450
 $EndSCHEMATC

Commit message: Updated copyright dates
Other:
- note added: "Design by Matt Weyland (HB9FRV)\nand Peter Klaentschi (HB9HY)\n\nBased on work by Tony Parks\n(c) 2017,18,19, CC-BY-SA"
- note removed: "Design by Matt Weyland (HB9FRV)\nand Peter Klaentschi (HB9HY)\n\nBased on work by Tony Parks\n(c) 2017, CC-BY-SA"
Changed lines of the file:
@@
 An SMD soldering practice kit for hams.
 Text Notes 8050 6250 0    118  ~ 0
-Design by Matt Weyland (HB9FRV)\nand Peter Klaentschi (HB9HY)\n\nBased on work by Tony Parks\n(c) 2017, CC-BY-SA
+Design by Matt Weyland (HB9FRV)\nand Peter Klaentschi (HB9HY)\n\nBased on work by Tony Parks\n(c) 2017,18,19, CC-BY-SA
 Wire Wire Line
 	4850 4800 5250 4800

Commit message: Replaced footprints with versions from new kicad footprint library
Parts:
- added J?: I/Q Out, symbol Connector_Generic:Conn_01x03
- C1, C10, C11, C12, C13, C14, C16, C2, C3, C4, C5, C7, C9: footprint Capacitors_SMD:C_1206_HandSoldering -> Capacitor_SMD:C_1206_3216Metric_Pad1.42x1.75mm_HandSolder
- D1, D2, D3, D4: footprint LEDs:LED_0805 -> LED_SMD:LED_0805_2012Metric_Pad1.15x1.40mm_HandSolder
- R1, R10, R2, R3, R4, R5, R6, R7, R8, R9: footprint Resistors_SMD:R_1206_HandSoldering -> Resistor_SMD:R_1206_3216Metric_Pad1.42x1.75mm_HandSolder
- R11, R12, R13, R14: footprint Resistors_SMD:R_0805_HandSoldering -> Resistor_SMD:R_1206_3216Metric_Pad1.42x1.75mm_HandSolder
- U3: footprint TO_SOT_Packages_SMD:SOT-89-3_Handsoldering -> Package_TO_SOT_SMD:SOT-89-3_Handsoldering
Connections:
- wire segments 136 -> 140

Commit message: Adding pin header for IQ audio tap
Parts:
- J5: renamed from J?; footprint (none) -> Connector_PinHeader_2.54mm:PinHeader_1x03_P2.54mm_Vertical
Connections:
- wire segments 140 -> 143
Changed lines of the file:
@@
 	9350 3100 9050 3100
 Connection ~ 9350 2900
-Wire Wire Line
-	10400 3650 10400 2700
 Connection ~ 9350 2250
 Connection ~ 9350 3650
@@
 $EndComp
 Wire Wire Line
-	10400 2250 10200 2250
-Wire Wire Line
 	9850 3650 9750 3650
 Wire Wire Line
@@
 Connection ~ 2150 2450
 $Comp
-L Connector_Generic:Conn_01x03 J?
+L Connector_Generic:Conn_01x03 J5
 U 1 1 5C938B4E
-P 10000 2700
-F 0 "J?" H 9920 2467 50  0000 C CNN
-F 1 "I/Q Out" H 9920 2466 50  0001 C CNN
-F 2 "" H 10000 2700 50  0001 C CNN
-F 3 "~" H 10000 2700 50  0001 C CNN
-	1    10000 2700
-	-1   0    0    1
-$EndComp
-Wire Wire Line
-	10200 2600 10200 2250
-Connection ~ 10200 2250
-Wire Wire Line
-	10200 2250 10150 2250
-Wire Wire Line
-	10200 2700 10400 2700
-Connection ~ 10400 2700
-Wire Wire Line
-	10400 2700 10400 2350
-$Comp
-L power:GND #PWR?
+P 10000 2900
+F 0 "J5" H 9920 2667 50  0000 C CNN
+F 1 "I/Q Out" H 9920 2666 50  0001 C CNN
+F 2 "Connector_PinHeader_2.54mm:PinHeader_1x03_P2.54mm_Vertical" H 10000 2900 50  0001 C CNN
+F 3 "~" H 10000 2900 50  0001 C CNN
+	1    10000 2900
+	-1   0    0    -1
+$EndComp
+$Comp
+L power:GND #PWR0101
 U 1 1 5C943FB5
-P 10200 2800
-F 0 "#PWR?" H 10200 2550 50  0001 C CNN
-F 1 "GND" H 10205 2627 50  0000 C CNN
-F 2 "" H 10200 2800 50  0001 C CNN
-F 3 "" H 10200 2800 50  0001 C CNN
-	1    10200 2800
-	1    0    0    -1
-$EndComp
+P 10000 2500
+F 0 "#PWR0101" H 10000 2250 50  0001 C CNN
+F 1 "GND" H 10005 2327 50  0000 C CNN
+F 2 "" H 10000 2500 50  0001 C CNN
+F 3 "" H 10000 2500 50  0001 C CNN
+	1    10000 2500
+	-1   0    0    -1
+$EndComp
+Wire Wire Line
+	10400 2350 10400 3000
+Wire Wire Line
+	10150 2250 10300 2250
+Wire Wire Line
+	10000 2500 10200 2500
+Wire Wire Line
+	10200 2500 10200 2800
+Wire Wire Line
+	10200 3000 10400 3000
+Connection ~ 10400 3000
+Wire Wire Line
+	10400 3000 10400 3650
+Wire Wire Line
+	10200 2900 10300 2900
+Wire Wire Line
+	10300 2900 10300 2250
+Connection ~ 10300 2250
+Wire Wire Line
+	10300 2250 10400 2250
 $EndSCHEMATC

Commit message: Replaced connector footprints with versions from new kicad footprint library
Parts:
- J3: footprint Pin_Headers:Pin_Header_Straight_2x03_Pitch2.54mm -> Connector_PinHeader_2.54mm:PinHeader_2x03_P2.54mm_Vertical
- J4: footprint Pin_Headers:Pin_Header_Straight_1x03_Pitch2.54mm -> Connector_PinHeader_2.54mm:PinHeader_1x03_P2.54mm_Vertical
- J8: footprint Pin_Headers:Pin_Header_Angled_1x05_Pitch2.54mm -> Connector_PinHeader_2.54mm:PinHeader_1x05_P2.54mm_Horizontal
Changed lines of the file:
@@
 F 0 "J3" H 4550 7167 50  0000 C CNN
 F 1 "ISP" H 4550 7076 50  0000 C CNN
-F 2 "Pin_Headers:Pin_Header_Straight_2x03_Pitch2.54mm" H 4500 6850 50  0001 C CNN
+F 2 "Connector_PinHeader_2.54mm:PinHeader_2x03_P2.54mm_Vertical" H 4500 6850 50  0001 C CNN
 F 3 "" H 4500 6850 50  0001 C CNN
 F 4 "DIST DIGIKEY 609-2846-ND" H 4500 6850 50  0001 C CNN "BOM"
@@
 F 0 "J8" H 920 3475 50  0000 C CNN
 F 1 "PWR" H 920 3566 50  0000 C CNN
-F 2 "Pin_Headers:Pin_Header_Angled_1x05_Pitch2.54mm" H 1000 3900 50  0001 C CNN
+F 2 "Connector_PinHeader_2.54mm:PinHeader_1x05_P2.54mm_Horizontal" H 1000 3900 50  0001 C CNN
 F 3 "" H 1000 3900 50  0001 C CNN
 F 4 "DIST DIGIKEY  S1012EC-05-ND" H 1000 3900 50  0001 C CNN "BOM"
@@
 F 0 "J4" H 8019 3825 50  0000 C CNN
 F 1 "LO" H 8019 3916 50  0000 C CNN
-F 2 "Pin_Headers:Pin_Header_Straight_1x03_Pitch2.54mm" H 8100 4150 50  0001 C CNN
+F 2 "Connector_PinHeader_2.54mm:PinHeader_1x03_P2.54mm_Vertical" H 8100 4150 50  0001 C CNN
 F 3 "~" H 8100 4150 50  0001 C CNN
 	1    8100 4150

Commit message: Adding missing BOM fields
Parts:
- J2: BOM (none) -> CON-SMA-EDGE-S-ND
Changed lines of the file:
@@
 F 2 "local:SMA_edge_mount_small" H 1000 2450 50  0001 C CNN
 F 3 "" H 1000 2450 50  0001 C CNN
+F 4 " CON-SMA-EDGE-S-ND " H 1000 2450 50  0001 C CNN "BOM"
 	1    1000 2450
 	-1   0    0    -1
@@
 U 1 1 5C938B4E
 P 10000 2900
-F 0 "J5" H 9920 2667 50  0000 C CNN
+F 0 "J5" H 10150 2900 50  0000 C CNN
 F 1 "I/Q Out" H 9920 2666 50  0001 C CNN
 F 2 "Connector_PinHeader_2.54mm:PinHeader_1x03_P2.54mm_Vertical" H 10000 2900 50  0001 C CNN

Commit message: Bumping version to 1.2 on schematic and PCB
Other:
- note added: "OMSDR Rev. 1.2"
- note removed: "OMSDR Rev. 1.1"
Changed lines of the file:
@@
 	7750 4050 7750 4900
 Text Notes 750  1050 0    295  ~ 59
-OMSDR Rev. 1.1
+OMSDR Rev. 1.2
 Text Notes 4700 1050 0    197  ~ 39
 An SMD soldering practice kit for hams.
