File: omsdr.sch (KiCad schematic (older format))
At the start: 54 parts, among them J1 I/Q Out, J2 ANT, J3 ISP, J4 LO, J5 I/Q Out, J8 PWR, SW1 SW_SPST, SW2 SW_SPST, T1 CX2074NL, U1 LT6231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

Commit message: New copyright owners for 1.2 version of the project.
Other:
- note added: "Design by Matt Weyland (HB9FRV)\n\nBased on work by Tony Parks\n(c) 2017,18,19, CC-BY-SA"
- note removed: "Design by Matt Weyland (HB9FRV)\nand Peter Klaentschi (HB9HY)\n\nBased on work by Tony Parks\n(c) 2017,18,19, CC-BY-SA"
Changed lines of the file:
@@
 An SMD soldering practice kit for hams.
 Text Notes 8050 6250 0    118  ~ 0
-Design by Matt Weyland (HB9FRV)\nand Peter Klaentschi (HB9HY)\n\nBased on work by Tony Parks\n(c) 2017,18,19, CC-BY-SA
+Design by Matt Weyland (HB9FRV)\n\nBased on work by Tony Parks\n(c) 2017,18,19, CC-BY-SA
 Wire Wire Line
 	4850 4800 5250 4800
