File: omsdr.kicad_sch (KiCad schematic)
At the start: 54 parts, among them J1 I/Q Out, J2 ANT, J3 ISP, J4 LO, J5 I/Q Out, J8 IO, SW1 SW_SPST, SW2 SW_SPST, T1 CX2074NL, U1 LT6231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

Commit message: Fixing BOM entry for SMA connector
Parts:
- J2: BOM CON-SMA-EDGE-S-ND -> DIST DIGIKEY CON-SMA-EDGE-S-ND
Changed lines of the file:
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@@
       (effects (font (size 1.27 1.27)) hide)
     )
-    (property "BOM" " CON-SMA-EDGE-S-ND " (id 4) (at 25.4 62.23 0)
+    (property "BOM" "DIST DIGIKEY CON-SMA-EDGE-S-ND " (id 4) (at 25.4 62.23 0)
       (effects (font (size 1.27 1.27)) hide)
     )

Commit message: Using crystal footprint from the KiCad library (pcb & 3d model)
Parts:
- X1: footprint Crystals:Crystal_SMD_HC49-SD -> Crystal:Crystal_SMD_HC49-SD
Changed lines of the file:
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@@
     (property "Reference" "X1" (id 0) (at 149.225 128.905 90))
     (property "Value" "25 MHz" (id 1) (at 146.685 131.445 90))
-    (property "Footprint" "Crystals:Crystal_SMD_HC49-SD" (id 2) (at 153.035 129.54 0)
+    (property "Footprint" "Crystal:Crystal_SMD_HC49-SD" (id 2) (at 153.035 129.54 0)
       (effects (font (size 1.27 1.27)) hide)
     )
@@
     )
     (path "/00000000-0000-0000-0000-00005a052ea0"
-      (reference "X1") (unit 1) (value "25 MHz") (footprint "Crystals:Crystal_SMD_HC49-SD")
-    )
-  )
+      (reference "X1") (unit 1) (value "25 MHz") (footprint "Crystal:Crystal_SMD_HC49-SD")
+    )
+  )

Commit message: Replacing push buttons with current kicad footprints and 3d models
Parts:
- SW1: value SW_SPST -> LEFT; footprint Buttons_Switches_SMD:SW_SPST_TL3342 -> Button_Switch_SMD:SW_SPST_TL3342
- SW2: value SW_SPST -> RIGHT; footprint Buttons_Switches_SMD:SW_SPST_TL3342 -> Button_Switch_SMD:SW_SPST_TL3342
Changed lines of the file:
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@@
     (in_bom yes) (on_board yes)
     (property "Reference" "SW1" (id 0) (at 152.4 164.211 0))
-    (property "Value" "SW_SPST" (id 1) (at 152.4 166.5224 0))
-    (property "Footprint" "Buttons_Switches_SMD:SW_SPST_TL3342" (id 2) (at 152.4 170.18 0)
+    (property "Value" "LEFT" (id 1) (at 152.4 166.5224 0))
+    (property "Footprint" "Button_Switch_SMD:SW_SPST_TL3342" (id 2) (at 152.4 170.18 0)
       (effects (font (size 1.27 1.27)) hide)
     )
@@
   (symbol (lib_id "Switch:SW_SPST") (at 152.4 177.8 0) (unit 1)
     (in_bom yes) (on_board yes)
-    (property "Reference" "SW2" (id 0) (at 152.4 171.831 0))
-    (property "Value" "SW_SPST" (id 1) (at 152.4 174.1424 0))
-    (property "Footprint" "Buttons_Switches_SMD:SW_SPST_TL3342" (id 2) (at 152.4 177.8 0)
+    (property "Reference" "SW2" (id 0) (at 152.4 180.975 0))
+    (property "Value" "RIGHT" (id 1) (at 152.4 183.515 0))
+    (property "Footprint" "Button_Switch_SMD:SW_SPST_TL3342" (id 2) (at 152.4 177.8 0)
       (effects (font (size 1.27 1.27)) hide)
     )
@@
     )
     (path "/00000000-0000-0000-0000-00005a06e759"
-      (reference "SW1") (unit 1) (value "SW_SPST") (footprint "Buttons_Switches_SMD:SW_SPST_TL3342")
+      (reference "SW1") (unit 1) (value "LEFT") (footprint "Button_Switch_SMD:SW_SPST_TL3342")
     )
     (path "/00000000-0000-0000-0000-00005a06e8b0"
-      (reference "SW2") (unit 1) (value "SW_SPST") (footprint "Buttons_Switches_SMD:SW_SPST_TL3342")
+      (reference "SW2") (unit 1) (value "RIGHT") (footprint "Button_Switch_SMD:SW_SPST_TL3342")
     )
     (path "/00000000-0000-0000-0000-00005a04a23a"
